File: LMN.kicad_pcb (KiCad board)
At the start: 2 copper layers, 304.8 x 95.2 mm, 100 parts, among them SW1 SW_Push, SW10 SW_Push, SW11 SW_Push, SW12 SW_Push, SW13 SW_Push, SW14 SW_Push, SW15 SW_Push, SW16 SW_Push, SW17 SW_Push, SW18 SW_Push, SW19 SW_Push, SW2 SW_Push, SW20 SW_Push, SW21 SW_Push, SW22 SW_Push, SW23 SW_Push, SW24 SW_Push, SW25 SW_Push, SW26 SW_Push, SW27 SW_Push, SW28 SW_Push, SW29 SW_Push, SW3 SW_Push, SW30 SW_Push, SW31 SW_Push, SW32 SW_Push, SW33 SW_Push, SW34 SW_Push, SW35 SW_Push, SW36 SW_Push, SW37 SW_Push, SW38 SW_Push, SW39 SW_Push, SW4 SW_Push, SW40 SW_Push, SW41 SW_Push, SW42 SW_Push, SW43 SW_Push, SW44 SW_Push, SW45 SW_Push, SW5 SW_Push, SW6 SW_Push, SW7 SW_Push, SW8 SW_Push, SW9 SW_Push, U1 EC11E_H20, U2 EC11E_H20, U3 EC11E_H20, U4 EC11E_H20, U5 COM-09032, U6 teensy_4.1

Commit message: Add mounting holes
Parts:
- added REF**: Mounting Hole, LMN:Mounting_Hole, F.Cu at (47.7, 104.7)
- added REF**: Mounting Hole, LMN:Mounting_Hole, F.Cu at (307.2, 38.1)
- added REF**: Mounting Hole, LMN:Mounting_Hole, F.Cu at (142.9, 76.2)
- added REF**: Mounting Hole, LMN:Mounting_Hole, F.Cu at (200.0, 76.2)
- added REF**: Mounting Hole, LMN:Mounting_Hole, F.Cu at (326.2, 95.2)
- added REF**: Mounting Hole, LMN:Mounting_Hole, F.Cu at (142.9, 38.1)
Changed lines of the file:
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@@
     )
+  )
+  (footprint "LMN:Mounting_Hole" (layer "F.Cu")
+    (at 47.71525 104.7115 90)
+    (attr through_hole)
+    (fp_text reference "REF**" (at 0 4.1 90 unlocked) (layer "F.SilkS") hide
+      (effects (font (size 1 1) (thickness 0.15)))
+    )
+    (fp_text value "Mounting Hole" (at 0 5.6 90 unlocked) (layer "F.Fab")
+      (effects (font (size 1 1) (thickness 0.15)))
+    )
+    (pad "" np_thru_hole oval (at 0 0 90) (size 5 2.54) (drill oval 5 2.54) (layers F&B.Cu *.Mask))
   )
   (footprint "Switch_Keyboard_Cherry_MX:SW_Cherry_MX_PCB_1.00u" (layer "F.Cu")
@@
       (rotate (xyz 0 -180 0))
     )
+  )
+  (footprint "LMN:Mounting_Hole" (layer "F.Cu")
+    (at 307.18125 38.1 90)
+    (attr through_hole)
+    (fp_text reference "REF**" (at 0 4.1 90 unlocked) (layer "F.SilkS") hide
+      (effects (font (size 1 1) (thickness 0.15)))
+    )
+    (fp_text value "Mounting Hole" (at 0 5.6 90 unlocked) (layer "F.Fab")
+      (effects (font (size 1 1) (thickness 0.15)))
+    )
+    (pad "" np_thru_hole oval (at 0 0 90) (size 5 2.54) (drill oval 5 2.54) (layers F&B.Cu *.Mask))
   )
   (footprint "Switch_Keyboard_Cherry_MX:SW_Cherry_MX_PCB_1.00u" (layer "F.Cu")
@@
     )
   )
+  (footprint "LMN:Mounting_Hole" (layer "F.Cu")
+    (at 142.875 76.2 90)
+    (attr through_hole)
+    (fp_text reference "REF**" (at 0 4.1 90 unlocked) (layer "F.SilkS") hide
+      (effects (font (size 1 1) (thickness 0.15)))
+    )
+    (fp_text value "Mounting Hole" (at 0 5.6 90 unlocked) (layer "F.Fab")
+      (effects (font (size 1 1) (thickness 0.15)))
+    )
+    (pad "" np_thru_hole oval (at 0 0 90) (size 5 2.54) (drill oval 5 2.54) (layers F&B.Cu *.Mask))
+  )
   (footprint "Switch_Keyboard_Cherry_MX:SW_Cherry_MX_PCB_1.00u" (layer "F.Cu")
     (at 190.5 76.2)
@@
     )
   )
+  (footprint "LMN:Mounting_Hole" (layer "F.Cu")
+    (at 200.025 76.2 90)
+    (attr through_hole)
+    (fp_text reference "REF**" (at 0 4.1 90 unlocked) (layer "F.SilkS") hide
+      (effects (font (size 1 1) (thickness 0.15)))
+    )
+    (fp_text value "Mounting Hole" (at 0 5.6 90 unlocked) (layer "F.Fab")
+      (effects (font (size 1 1) (thickness 0.15)))
+    )
+    (pad "" np_thru_hole oval (at 0 0 90) (size 5 2.54) (drill oval 5 2.54) (layers F&B.Cu *.Mask))
+  )
   (footprint "Switch_Keyboard_Cherry_MX:SW_Cherry_MX_PCB_1.00u" (layer "F.Cu")
     (at 209.55 114.3)
@@
       (rotate (xyz 0 0 0))
     )
+  )
+  (footprint "LMN:Mounting_Hole" (layer "F.Cu")
+    (at 326.23125 95.25 -90)
+    (attr through_hole)
+    (fp_text reference "REF**" (at 0 4.1 -90 unlocked) (layer "F.SilkS") hide
+      (effects (font (size 1 1) (thickness 0.15)))
+    )
+    (fp_text value "Mounting Hole" (at 0 5.6 -90 unlocked) (layer "F.Fab")
+      (effects (font (size 1 1) (thickness 0.15)))
+    )
+    (pad "" np_thru_hole oval (at 0 0 270) (size 5 2.54) (drill oval 5 2.54) (layers F&B.Cu *.Mask))
   )
   (footprint "Switch_Keyboard_Cherry_MX:SW_Cherry_MX_PCB_1.00u" (layer "F.Cu")
@@
     )
   )
-  (footprint "Switch_Keyboard_Cherry_MX:SW_Cherry_MX_PCB_1.00u" (layer "F.Cu")
+  (footprint "LMN:Mounting_Hole" (layer "F.Cu")
+    (at 142.875 38.1 90)
+    (attr through_hole)
+    (fp_text reference "REF**" (at 0 4.1 90 unlocked) (layer "F.SilkS") hide
+      (effects (font (size 1 1) (thickness 0.15)))
+    )
+    (fp_text value "Mounting Hole" (at 0 5.6 90 unlocked) (layer "F.Fab")
+      (effects (font (size 1 1) (thickness 0.15)))
+    )
+    (pad "" np_thru_hole oval (at 0 0 90) (size 5 2.54) (drill oval 5 2.54) (layers F&B.Cu *.Mask))
+  )
+  (footprint "Switch_Keyboard_Cherry_MX:SW_Cherry_MX_PCB_1.00u" (layer "F.Cu")
