File: LMN.kicad_pcb (KiCad board)
At the start: 2 copper layers, 304.8 x 95.2 mm, 106 parts, among them SW1 SW_Push, SW10 SW_Push, SW11 SW_Push, SW12 SW_Push, SW13 SW_Push, SW14 SW_Push, SW15 SW_Push, SW16 SW_Push, SW17 SW_Push, SW18 SW_Push, SW19 SW_Push, SW2 SW_Push, SW20 SW_Push, SW21 SW_Push, SW22 SW_Push, SW23 SW_Push, SW24 SW_Push, SW25 SW_Push, SW26 SW_Push, SW27 SW_Push, SW28 SW_Push, SW29 SW_Push, SW3 SW_Push, SW30 SW_Push, SW31 SW_Push, SW32 SW_Push, SW33 SW_Push, SW34 SW_Push, SW35 SW_Push, SW36 SW_Push, SW37 SW_Push, SW38 SW_Push, SW39 SW_Push, SW4 SW_Push, SW40 SW_Push, SW41 SW_Push, SW42 SW_Push, SW43 SW_Push, SW44 SW_Push, SW45 SW_Push, SW5 SW_Push, SW6 SW_Push, SW7 SW_Push, SW8 SW_Push, SW9 SW_Push, U1 EC11E_H20, U2 EC11E_H20, U3 EC11E_H20, U4 EC11E_H20, U5 COM-09032, U6 teensy_4.1

Commit message: Update gerbers
Parts:
- moved REF** 23.3 mm to (69.1, 95.2)
Changed lines of the file:
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@@
   )
   (footprint "LMN:Mounting_Hole" (layer "F.Cu")
-    (at 47.71525 104.7115 90)
+    (at 69.05625 95.25 90)
     (attr through_hole)
     (fp_text reference "REF**" (at 0 4.1 90 unlocked) (layer "F.SilkS") hide
@@
     (fp_line (start 9.525 -9.525) (end -9.525 -9.525) (layer "Dwgs.User") (width 0.1))
     (fp_line (start -9.525 -9.525) (end -9.525 9.525) (layer "Dwgs.User") (width 0.1))
-    (fp_line (start 9.525 9.525) (end 9.525 -9.525) (layer "Dwgs.User") (width 0.1))
     (fp_line (start -9.525 9.525) (end 9.525 9.525) (layer "Dwgs.User") (width 0.1))
+    (fp_line (start 9.525 9.525) (end 9.525 -9.525) (layer "Dwgs.User") (width 0.1))
     (fp_line (start 7 7) (end 7 -7) (layer "Eco1.User") (width 0.1))
     (fp_line (start 7 -7) (end -7 -7) (layer "Eco1.User") (width 0.1))
@@
   (gr_poly
     (pts
-      (xy 190.61678 95.408832)
-      (xy 190.620095 95.290556)
-      (xy 190.629932 95.173834)
-      (xy 190.646132 95.058809)
-      (xy 190.668534 94.945625)
-      (xy 190.696979 94.834427)
-      (xy 190.731307 94.725359)
-      (xy 190.771356 94.618566)
-      (xy 190.816968 94.514192)
-      (xy 190.867982 94.412382)
-      (xy 190.924239 94.31328)
-      (xy 190.985577 94.21703)
-      (xy 191.051838 94.123777)
-      (xy 191.122861 94.033665)
-      (xy 191.198485 93.946839)
-      (xy 191.278551 93.863443)
-      (xy 191.3629 93.783621)
-      (xy 191.45137 93.707518)
-      (xy 191.543801 93.635278)
-      (xy 191.640035 93.567046)
-      (xy 191.73991 93.502967)
-      (xy 191.843266 93.443183)
-      (xy 191.949944 93.387841)
-      (xy 192.059784 93.337084)
-      (xy 192.172624 93.291056)
-      (xy 192.288306 93.249903)
-      (xy 192.40667 93.213768)
-      (xy 192.527554 93.182797)
-      (xy 192.6508 93.157132)
-      (xy 192.776246 93.13692)
-      (xy 192.903734 93.122304)
-      (xy 193.033103 93.113428)
-      (xy 193.164192 93.110437)
-      (xy 193.295282 93.113428)
-      (xy 193.42465 93.122304)
-      (xy 193.552138 93.13692)
-      (xy 193.677585 93.157132)
-      (xy 193.80083 93.182797)
-      (xy 193.921715 93.213768)
-      (xy 194.040078 93.249903)
-      (xy 194.15576 93.291056)
-      (xy 194.268601 93.337084)
-      (xy 194.37844 93.387841)
-      (xy 194.485118 93.443183)
-      (xy 194.588474 93.502967)
-      (xy 194.688349 93.567046)
-      (xy 194.784583 93.635278)
-      (xy 194.877015 93.707518)
-      (xy 194.965485 93.783621)
-      (xy 195.049833 93.863443)
-      (xy 195.129899 93.946839)
-      (xy 195.205524 94.033665)
-      (xy 195.276546 94.123777)
-      (xy 195.342807 94.21703)
-      (xy 195.404145 94.31328)
-      (xy 195.460402 94.412382)
-      (xy 195.511416 94.514192)
-      (xy 195.557028 94.618566)
-      (xy 195.597078 94.725359)
-      (xy 195.631405 94.834427)
-      (xy 195.65985 94.945625)
-      (xy 195.682252 95.058809)
-      (xy 195.698452 95.173834)
-      (xy 195.70829 95.290556)
-      (xy 195.711604 95.408832)
-      (xy 195.70829 95.527106)
-      (xy 195.698452 95.643829)
-      (xy 195.682252 95.758854)
-      (xy 195.65985 95.872038)
-      (xy 195.631405 95.983236)
-      (xy 195.597078 96.092303)
-      (xy 195.557028 96.199096)
-      (xy 195.511416 96.30347)
-      (xy 195.460402 96.40528)
-      (xy 195.404145 96.504382)
-      (xy 195.342807 96.600632)
-      (xy 195.276546 96.693885)
-      (xy 195.205524 96.783997)
-      (xy 195.129899 96.870823)
-      (xy 195.049833 96.95422)
-      (xy 194.965485 97.034041)
-      (xy 194.877015 97.110144)
-      (xy 194.784583 97.182384)
-      (xy 194.688349 97.250616)
-      (xy 194.588474 97.314696)
-      (xy 194.485118 97.37448)
-      (xy 194.37844 97.429822)
-      (xy 194.268601 97.480579)
-      (xy 194.15576 97.526607)
-      (xy 194.040078 97.56776)
-      (xy 193.921715 97.603895)
-      (xy 193.80083 97.634867)
-      (xy 193.677585 97.660531)
-      (xy 193.552138 97.680744)
-      (xy 193.42465 97.69536)
-      (xy 193.295282 97.704236)
-      (xy 193.164192 97.707226)
-      (xy 193.033103 97.704236)
-      (xy 192.903734 97.69536)
-      (xy 192.776246 97.680744)
-      (xy 192.6508 97.660531)
-      (xy 192.527554 97.634867)
-      (xy 192.40667 97.603895)
-      (xy 192.288306 97.56776)
-      (xy 192.172624 97.526607)
-      (xy 192.059784 97.480579)
-      (xy 191.949944 97.429822)
-      (xy 191.843266 97.37448)
-      (xy 191.73991 97.314696)
-      (xy 191.640035 97.250616)
-      (xy 191.543801 97.182384)
-      (xy 191.45137 97.110144)
-      (xy 191.3629 97.034041)
-      (xy 191.278551 96.95422)
-      (xy 191.198485 96.870823)
-      (xy 191.122861 96.783997)
-      (xy 191.051838 96.693885)
-      (xy 190.985577 96.600632)
-      (xy 190.924239 96.504382)
-      (xy 190.867982 96.40528)
-      (xy 190.816968 96.30347)
-      (xy 190.771356 96.199096)
-      (xy 190.731307 96.092303)
-      (xy 190.696979 95.983236)
-      (xy 190.668534 95.872038)
-      (xy 190.646132 95.758854)
-      (xy 190.629932 95.643829)
-      (xy 190.620095 95.527106)
-      (xy 190.61678 95.408832)
-    ) (layer "F.Mask") (width 0.105833) (fill solid))
-  (gr_poly
-    (pts
       (xy 151.26453 95.250002)
       (xy 151.253537 95.590026)
@@
       (xy 280.554596 95.39655)
     ) (layer "F.Mask") (width 0.105833) (fill solid))
+  (gr_poly
+    (pts
+      (xy 190.61678 95.408832)
+      (xy 190.620095 95.290556)
+      (xy 190.629932 95.173834)
+      (xy 190.646132 95.058809)
+      (xy 190.668534 94.945625)
+      (xy 190.696979 94.834427)
+      (xy 190.731307 94.725359)
+      (xy 190.771356 94.618566)
+      (xy 190.816968 94.514192)
+      (xy 190.867982 94.412382)
+      (xy 190.924239 94.31328)
+      (xy 190.985577 94.21703)
+      (xy 191.051838 94.123777)
+      (xy 191.122861 94.033665)
+      (xy 191.198485 93.946839)
+      (xy 191.278551 93.863443)
+      (xy 191.3629 93.783621)
+      (xy 191.45137 93.707518)
+      (xy 191.543801 93.635278)
+      (xy 191.640035 93.567046)
+      (xy 191.73991 93.502967)
+      (xy 191.843266 93.443183)
+      (xy 191.949944 93.387841)
+      (xy 192.059784 93.337084)
+      (xy 192.172624 93.291056)
+      (xy 192.288306 93.249903)
+      (xy 192.40667 93.213768)
+      (xy 192.527554 93.182797)
+      (xy 192.6508 93.157132)
+      (xy 192.776246 93.13692)
+      (xy 192.903734 93.122304)
+      (xy 193.033103 93.113428)
+      (xy 193.164192 93.110437)
+      (xy 193.295282 93.113428)
+      (xy 193.42465 93.122304)
+      (xy 193.552138 93.13692)
+      (xy 193.677585 93.157132)
+      (xy 193.80083 93.182797)
+      (xy 193.921715 93.213768)
+      (xy 194.040078 93.249903)
+      (xy 194.15576 93.291056)
+      (xy 194.268601 93.337084)
+      (xy 194.37844 93.387841)
+      (xy 194.485118 93.443183)
+      (xy 194.588474 93.502967)
+      (xy 194.688349 93.567046)
+      (xy 194.784583 93.635278)
+      (xy 194.877015 93.707518)
+      (xy 194.965485 93.783621)
+      (xy 195.049833 93.863443)
+      (xy 195.129899 93.946839)
+      (xy 195.205524 94.033665)
+      (xy 195.276546 94.123777)
+      (xy 195.342807 94.21703)
+      (xy 195.404145 94.31328)
+      (xy 195.460402 94.412382)
+      (xy 195.511416 94.514192)
+      (xy 195.557028 94.618566)
+      (xy 195.597078 94.725359)
+      (xy 195.631405 94.834427)
+      (xy 195.65985 94.945625)
+      (xy 195.682252 95.058809)
+      (xy 195.698452 95.173834)
+      (xy 195.70829 95.290556)
+      (xy 195.711604 95.408832)
+      (xy 195.70829 95.527106)
+      (xy 195.698452 95.643829)
+      (xy 195.682252 95.758854)
+      (xy 195.65985 95.872038)
+      (xy 195.631405 95.983236)
+      (xy 195.597078 96.092303)
+      (xy 195.557028 96.199096)
+      (xy 195.511416 96.30347)
+      (xy 195.460402 96.40528)
+      (xy 195.404145 96.504382)
+      (xy 195.342807 96.600632)
+      (xy 195.276546 96.693885)
+      (xy 195.205524 96.783997)
+      (xy 195.129899 96.870823)
+      (xy 195.049833 96.95422)
+      (xy 194.965485 97.034041)
+      (xy 194.877015 97.110144)
+      (xy 194.784583 97.182384)
+      (xy 194.688349 97.250616)
+      (xy 194.588474 97.314696)
+      (xy 194.485118 97.37448)
+      (xy 194.37844 97.429822)
+      (xy 194.268601 97.480579)
+      (xy 194.15576 97.526607)
+      (xy 194.040078 97.56776)
+      (xy 193.921715 97.603895)
+      (xy 193.80083 97.634867)
+      (xy 193.677585 97.660531)
+      (xy 193.552138 97.680744)
+      (xy 193.42465 97.69536)
+      (xy 193.295282 97.704236)
+      (xy 193.164192 97.707226)
+      (xy 193.033103 97.704236)
+      (xy 192.903734 97.69536)
+      (xy 192.776246 97.680744)
+      (xy 192.6508 97.660531)
+      (xy 192.527554 97.634867)
+      (xy 192.40667 97.603895)
+      (xy 192.288306 97.56776)
+      (xy 192.172624 97.526607)
+      (xy 192.059784 97.480579)
+      (xy 191.949944 97.429822)
+      (xy 191.843266 97.37448)
+      (xy 191.73991 97.314696)
+      (xy 191.640035 97.250616)
+      (xy 191.543801 97.182384)
+      (xy 191.45137 97.110144)
+      (xy 191.3629 97.034041)
+      (xy 191.278551 96.95422)
+      (xy 191.198485 96.870823)
+      (xy 191.122861 96.783997)
+      (xy 191.051838 96.693885)
+      (xy 190.985577 96.600632)
+      (xy 190.924239 96.504382)
+      (xy 190.867982 96.40528)
+      (xy 190.816968 96.30347)
+      (xy 190.771356 96.199096)
+      (xy 190.731307 96.092303)
+      (xy 190.696979 95.983236)
+      (xy 190.668534 95.872038)
+      (xy 190.646132 95.758854)
+      (xy 190.629932 95.643829)
+      (xy 190.620095 95.527106)
+      (xy 190.61678 95.408832)
+    ) (layer "F.Mask") (width 0.105833) (fill solid))
   (gr_line (start 31.100265 102.2497) (end 31.100265 88.2504) (layer "Dwgs.User") (width 0.05))
   (gr_line (start 154.925235 88.2504) (end 168.924235 88.2504) (layer "Dwgs.User") (width 0.05))
@@
     )
   )
-  (group "" (id fb61a683-83da-47d7-a930-042655a2d475)
-    (members
-      1400b28e-0ae9-49ae-b232-acc149de5fa7
-      41dfcb4b-4be6-46cc-bd52-5a4ae84f1893
-      42ff67e1-2f56-4a19-81d1-e5f22a2b9110
-    )
-  )
